File: CAO/DRAGSTER/DRAGSTER.kicad_pcb (KiCad board)
At the start: 4 copper layers, 60 x 60 mm, 47 parts, among them J1 ESC, J2 BLUETOOTH, J3 ACCELEROMETER, J4 Conn_02x07_Odd_Even, J5 Conn_01x16_Socket, Q1 AO3401A, SW1 SW_Push, SW2 SW_Push, U1 STM32G431CBUx, U2 LMR51625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

Commit message: updated pcb
Parts:
- added G***: LOGO, Custom_Library:img, F.Cu at (187.8, 79.8)
- moved TP1 9.97 mm to (187.4, 88.0)
- moved L2 3.19 mm to (171.6, 89.6)
- moved C19 2.78 mm to (182.2, 90.6), turned to -90 degrees
Routing:
- net +5V: track 101.5 -> 30.7 mm, vias 2 -> 16
- net GND: track 64.6 -> 51.9 mm, vias 51 -> 47
- net +3.3V: track 75.6 -> 68.3 mm, vias 28 -> 30
- net SW: track 11.9 -> 9.99 mm
- added copper zone on In2.Cu, net +5V
Other:
- board text added: "ACCEL"
- board text added: "B"
- board text added: "BOOT"
- board text added: "BT"
- board text added: "NRST"
- board text added: "SCREEN"
- board text added: "SWD"
- board text added: "T"
- board text added: "T.KOYAZANDE"
