File: CAO/DRAGSTER_KICAD/DRAGSTER.kicad_sch (KiCad schematic)
At the start: 47 parts, among them J1 ESC, J2 BLUETOOTH, J3 ACCELEROMETER, J4 Conn_02x07_Odd_Even, J5 Conn_01x16_Socket, Q1 AO3401A, SW1 SW_Push, SW2 SW_Push, U1 STM32G431CBUx, U2 LMR51625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

Commit message: reshuffled stuffs a bit
Parts:
- removed C8: 1u, Capacitor_SMD:C_0402_1005Metric_Pad0.74x0.62mm_HandSolder, symbol Device:C_Small
- removed F1: 350mA, Fuse:Fuse_0402_1005Metric_Pad0.77x0.64mm_HandSolder, symbol Device:Polyfuse_Small
- removed FB1: 600 @ 600MHz, Inductor_SMD:L_0402_1005Metric_Pad0.77x0.64mm_HandSolder, symbol Device:FerriteBead_Small
- removed H2, H4: MountingHole_Pad, MountingHole:MountingHole_4.3mm_M4_Pad_Via, symbol Mechanical:MountingHole_Pad
- removed J2: BLUETOOTH, Connector_PinSocket_2.00mm:PinSocket_1x05_P2.00mm_Horizontal, symbol Connector:Conn_01x05_Socket
- removed L1: 39n, Inductor_SMD:L_0402_1005Metric_Pad0.77x0.64mm_HandSolder, symbol Device:L_Small
- added J6: Conn_01x06_Socket, Connector_PinSocket_2.54mm:PinSocket_1x06_P2.54mm_Horizontal, symbol Connector:Conn_01x06_Socket
- added R4, R5: 4k7, Resistor_SMD:R_0402_1005Metric_Pad0.72x0.64mm_HandSolder, symbol Device:R_Small
- added SW3: SW_Push, Custom_Library:15715636, symbol Switch:SW_Push
- C1: value 1u -> 100n; MPN GXT155R60J105KE01D -> 04026C104MAT2A
- C2: value 10n -> 100n; MPN GRM155R70J103KA01D -> 04026C104MAT2A
- D2: footprint LED_SMD:LED_WS2812B-2020_PLCC4_2.0x2.0mm -> LED_SMD:LED_WS2812B_PLCC4_5.0x5.0mm_P3.2mm
- J4: footprint Connector_PinHeader_2.54mm:PinHeader_2x07_P2.54mm_Vertical_SMD -> Custom_Library:FTSH-107-XX-YYY-DV-K
- J5: footprint Connector_PinSocket_2.00mm:PinSocket_1x16_P2.00mm_Vertical -> Connector_PinSocket_2.54mm:PinSocket_1x16_P2.54mm_Vertical
Connections:
- net +3.3V: now also C2.1, U1.21 (VDDA), R4.2, R5.2
- net +5V: now also J6.2 (Pin_2)
- net GND: now also C1.1, J6.3 (Pin_3), SW3.1; no longer C1.2
- net I2C_SCL: now also R4.1
- net I2C_SDA: now also R5.1
- net KEY_BLUETOOTH: now also J6.1 (Pin_1)
- net USART2_RX: now also J6.4 (Pin_4)
- net USART2_TX: now also J6.5 (Pin_5)
- net VIN: now also Q1.2 (S)
- net USER_BUTTON: now reaches U1.12 (PA4)
- net USER_BUTTON: now also C1.2, SW3.2
- net PWM_LED_DATA_IN: now reaches U1.24 (PB11)
- net PWM_LED_DATA_IN: now also D2.3 (DIN)
- removed net +3.3VA: C1.1, C2.1, U1.21 (VDDA)
- net LED_DATA_IN: no longer names the net of U1.16 (PC4)
- net LED_DATA_IN: no longer D2.3 (DIN)
Other:
- moved on the sheet: C16, C19, C9, TP1
